File: hw/switch.kicad_pcb (KiCad board)
At the start: 2 copper layers, 25.4 x 12.7 mm, 14 parts, among them IC1 MSP430FR2000IPW16, J1 Conn_01x02, J2 Conn_01x03, J3 Conn_01x03, J4 Conn_01x02, Q1 2SK2231, U1 AP2112K-3.3

Commit message: repo name
Other:
- board text added: "github.com/ondrejh/rc_switch"

Commit message: bom
Parts:
- C1, C2: value C_Small -> 220n
- R1: value R_Small -> 10k
- R2: value R_Small -> 22k
- R3: value R_Small -> 1k0
- U1: value AP2112K-3.3 -> AP2202K-3.3
Changed lines of the file:
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@@
     (visible_elements FFFFFF7F)
     (pcbplotparams
-      (layerselection 0x010fc_ffffffff)
+      (layerselection 0x010e0_ffffffff)
       (usegerberextensions false)
       (usegerberattributes true)
@@
       (outputformat 1)
       (mirror false)
-      (drillshape 1)
+      (drillshape 0)
       (scaleselection 1)
       (outputdirectory ""))
@@
       (effects (font (size 1 1) (thickness 0.15)))
     )
-    (fp_text value AP2112K-3.3 (at 0 2.9 90) (layer F.Fab)
+    (fp_text value AP2202K-3.3 (at 0 2.9 90) (layer F.Fab)
       (effects (font (size 1 1) (thickness 0.15)))
     )
@@
       (effects (font (size 1 1) (thickness 0.15)))
     )
-    (fp_text value R_Small (at 0 1.43) (layer F.Fab)
+    (fp_text value 10k (at 0 1.43) (layer F.Fab)
       (effects (font (size 1 1) (thickness 0.15)))
     )
@@
       (effects (font (size 1 1) (thickness 0.15)))
     )
-    (fp_text value R_Small (at 0 1.43) (layer F.Fab)
+    (fp_text value 22k (at 0 1.43) (layer F.Fab)
       (effects (font (size 1 1) (thickness 0.15)))
     )
@@
       (effects (font (size 1 1) (thickness 0.15)) (justify mirror))
     )
-    (fp_text value R_Small (at 0 -1.43) (layer B.Fab)
+    (fp_text value 1k0 (at 0 -1.43) (layer B.Fab)
       (effects (font (size 1 1) (thickness 0.15)) (justify mirror))
     )
@@
       (effects (font (size 1 1) (thickness 0.15)))
     )
-    (fp_text value C_Small (at 0 1.68 90) (layer F.Fab)
+    (fp_text value 220n (at 0 1.68 90) (layer F.Fab)
       (effects (font (size 1 1) (thickness 0.15)))
     )
@@
       (effects (font (size 1 1) (thickness 0.15)))
     )
-    (fp_text value C_Small (at 0 1.68 90) (layer F.Fab)
+    (fp_text value 220n (at 0 1.68 90) (layer F.Fab)
       (effects (font (size 1 1) (thickness 0.15)))
     )
@@
   (segment (start 148.9025 88.605) (end 146.71 88.605) (width 0.35) (layer F.Cu) (net 2))
   (segment (start 140.335 86.68) (end 140.335 85.09) (width 0.35) (layer F.Cu) (net 2))
-  (via (at 139.7 85.09) (size 0.8) (drill 0.4) (layers F.Cu B.Cu) (net 2))
+  (via (at 139.7 85.09) (size 0.8) (drill 0.4) (layers F.Cu B.Cu) (net 2) (status 1000000))
   (segment (start 140.335 85.09) (end 139.7 85.09) (width 0.35) (layer F.Cu) (net 2))
   (segment (start 137.795 85.09) (end 139.7 85.09) (width 2.5) (layer B.Cu) (net 2))

Commit message: bom update
Parts:
- Q1: value 2SK2231 -> DMG4800LK3-13
- R1: value 10k -> 12k
Changed lines of the file:
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@@
       (effects (font (size 1 1) (thickness 0.15)) (justify mirror))
     )
-    (fp_text value 2SK2231 (at 0 -4.5) (layer B.Fab)
+    (fp_text value DMG4800LK3-13 (at 0 -4.5) (layer B.Fab)
       (effects (font (size 1 1) (thickness 0.15)) (justify mirror))
     )
@@
       (effects (font (size 1 1) (thickness 0.15)))
     )
-    (fp_text value 10k (at 0 1.43) (layer F.Fab)
+    (fp_text value 12k (at 0 1.43) (layer F.Fab)
       (effects (font (size 1 1) (thickness 0.15)))
     )
