File: hw/switch.sch (KiCad schematic (older format))
At the start: 14 parts, among them IC1 MSP430FR2000IPW16, J1 Conn_01x02, J2 Conn_01x03, J3 Conn_01x03, J4 Conn_01x02, Q1 2SK2231, U1 AP2112K-3.3

Commit message: bom
Parts:
- U1: value AP2112K-3.3 -> AP2202K-3.3
Changed lines of the file:
@@
 P 3800 3800
 F 0 "U1" H 3800 4142 50  0000 C CNN
-F 1 "AP2112K-3.3" H 3800 4051 50  0000 C CNN
+F 1 "AP2202K-3.3" H 3800 4051 50  0000 C CNN
 F 2 "Package_TO_SOT_SMD:SOT-23-5" H 3800 4125 50  0001 C CNN
 F 3 "https://www.diodes.com/assets/Datasheets/AP2112.pdf" H 3800 3900 50  0001 C CNN

Commit message: bom update
Parts:
- Q1: value 2SK2231 -> DMG4800LK3-13
- R1: value 10k -> 12k
Changed lines of the file:
@@
 P 2500 4200
 F 0 "R1" H 2559 4246 50  0000 L CNN
-F 1 "10k" H 2559 4155 50  0000 L CNN
+F 1 "12k" H 2559 4155 50  0000 L CNN
 F 2 "Resistor_SMD:R_0603_1608Metric" H 2500 4200 50  0001 C CNN
 F 3 "~" H 2500 4200 50  0001 C CNN
@@
 P 8900 3200
 F 0 "Q1" V 9242 3200 50  0000 C CNN
-F 1 "2SK2231" V 9151 3200 50  0000 C CNN
+F 1 "DMG4800LK3-13" V 9151 3200 50  0000 C CNN
 F 2 "Package_TO_SOT_SMD:TO-252-3_TabPin2" H 9100 3300 50  0001 C CNN
 F 3 "~" H 8900 3200 50  0001 C CNN
